Commit message: Changed files loading location to med_uav_description

File: urdf/windmill.base.urdf.xacro (robot description, xacro)
@@ -18,5 +18,5 @@
         <origin xyz="0 0 0" rpy="0 0 0" />
         <geometry>
-          <mesh filename="package://mmuav_description/meshes/windmill_base.dae"
+          <mesh filename="package://med_uav_description/meshes/windmill_base.dae"
             scale="2 2 2" />
         </geometry>
@@ -25,5 +25,5 @@
         <origin xyz="0 0 0" rpy="0 0 0"/>
         <geometry>
-          <mesh filename="package://mmuav_description/meshes/windmill_base.dae"
+          <mesh filename="package://med_uav_description/meshes/windmill_base.dae"
             scale="1 1 1" />
         </geometry>
@@ -45,5 +45,5 @@
         <origin xyz="0.16228 -0.00566 0.1" rpy="0 0 0" />
         <geometry>
-          <mesh filename="package://mmuav_description/meshes/windmill_rotor.dae"
+          <mesh filename="package://med_uav_description/meshes/windmill_rotor.dae"
             scale="2 2 2" />
         </geometry>
@@ -52,5 +52,5 @@
         <origin xyz="0 0 0" rpy="0 0 0"/>
         <geometry>
-          <mesh filename="package://mmuav_description/meshes/windmill_rotor.dae"
+          <mesh filename="package://med_uav_description/meshes/windmill_rotor.dae"
             scale="1 1 1" />
         </geometry>

File: urdf/windmill.gazebo.xacro (robot description, xacro)
@@ -15,5 +15,5 @@
   <xacro:property name="bag_file" value="windmill.bag" />
   <!-- Instantiate mmuav "mechanics" -->
-  <xacro:include filename="$(find mmuav_description)/urdf/windmill.base.urdf.xacro" />
+  <xacro:include filename="$(find med_uav_description)/urdf/windmill.base.urdf.xacro" />
   <xacro:include filename="$(find rotors_description)/urdf/component_snippets.xacro" />
 </robot>
