Commit message: added 1D laser

File: urdf/ardrone.urdf.xacro (robot description, xacro)
@@ -3,5 +3,5 @@
   <xacro:property name="namespace" value="$(arg namespace)" />
   <!-- Instantiate ardrone "mechanics" -->
-  	<xacro:include filename="$(find urs_ardrone_description)/urdf/ardrone_base.urdf.xacro" />
+  	<xacro:include filename="$(find med_uav_description)/urdf/ardrone_base.urdf.xacro" />
   	<xacro:include filename="$(find rotors_description)/urdf/component_snippets.xacro" />
 	<xacro:odometry_plugin_macro
@@ -34,3 +34,51 @@
 		<origin xyz="0.0 0.0 0.0" rpy="0.0 0.0 0.0" />
 	</xacro:odometry_plugin_macro>
+    <link name="laser1D_link">
+      <inertial>
+        <mass value="1e-5" />
+        <origin xyz="0 0 0" rpy="0 0 0"/>
+        <inertia ixx="1e-6" ixy="0" ixz="0" iyy="1e-6" iyz="0" izz="1e-6" />
+      </inertial>
+    </link>
+    <joint name="laser1D_joint" type="fixed">
+      <!--<axis xyz="0 0 1" />-->
+      <origin xyz="0.19 0 0.031" rpy="0 0 0"/>
+      <parent link="base_link"/>
+      <child link="laser1D_link"/>
+    </joint>
+ 	<gazebo reference="laser1D_link">
+		<sensor type="ray" name="laser1D_sensor">
+	      <pose>0 0 0 0 0 0</pose>
+	      <visualize>true</visualize>
+	      <update_rate>40</update_rate>
+	      <ray>
+	        <scan>
+	          <horizontal>
+	            <samples>1</samples>
+	            <resolution>1</resolution>
+	            <min_angle>0</min_angle>
+	            <max_angle>0</max_angle>
+	          </horizontal>
+	        </scan>
+	        <range>
+	          <min>0.10</min>
+	          <max>30.0</max>
+	          <resolution>0.01</resolution>
+	        </range>
+	        <noise>
+	          <type>gaussian</type>
+	          <!-- Noise parameters based on published spec for Hokuyo laser
+	               achieving "+-30mm" accuracy at range < 10m.  A mean of 0.0m and
+	               stddev of 0.01m will put 99.7% of samples within 0.03m of the true
+	               reading. -->
+	          <mean>0.0</mean>
+	          <stddev>0.01</stddev>
+	        </noise>
+	      </ray>
+	      <plugin name="gazebo_ros_head_hokuyo_controller" filename="libgazebo_ros_laser.so">
+	        <topicName>laser/scan</topicName>
+	        <frameName>laser1D_link</frameName>
+	      </plugin>
+	    </sensor>
+  	</gazebo>
 </robot>

File: urdf/ardrone_base.urdf.xacro (robot description, xacro)
@@ -35,5 +35,5 @@
   </xacro:property>
   <!-- Included URDF Files -->
-  <xacro:include filename="$(find urs_ardrone_description)/urdf/multirotor_base.urdf.xacro" />
+  <xacro:include filename="$(find med_uav_description)/urdf/multirotor_base.urdf.xacro" />
   <!-- Instantiate multirotor_base_macro once -->
   <xacro:multirotor_base_macro

File: urdf/multirotor_base.urdf.xacro (robot description, xacro)
@@ -19,5 +19,5 @@
         <origin xyz="0.055 0 0" rpy="0 0 -1.57079632679" />
         <geometry>
-          <mesh filename="package://urs_ardrone_description/meshes/${mesh_file}"
+          <mesh filename="package://med_uav_description/meshes/${mesh_file}"
             scale="0.001 0.001 0.001" />
           <!-- <box size="${body_width} ${body_width} ${body_height}"/> --> <!-- [m] [m] [m] -->
@@ -78,5 +78,5 @@
         <geometry>
           <!-- <cylinder length="0.005" radius="${radius_rotor}"/> --> <!-- [m] -->
-          <mesh filename="package://urs_ardrone_description/meshes/propeller_${direction}.dae"
+          <mesh filename="package://med_uav_description/meshes/propeller_${direction}.dae"
             scale="0.0008 0.0008 0.0008" />
           <!-- <box size="${2*radius_rotor} 0.01 0.005"/> -->

File: urdf/windmill.base.urdf.xacro (robot description, xacro)
@@ -22,11 +22,11 @@
         </geometry>
       </visual>
-      <!--collision name='collision'>
+      <collision name='collision'>
         <origin xyz="0 0 0" rpy="0 0 0"/>
         <geometry>
           <mesh filename="package://med_uav_description/meshes/windmill_base.dae"
-            scale="1 1 1" />
+            scale="2 2 2" />
         </geometry>
-      </collision-->
+      </collision>
     </link>
     <!--_____________________________________________________________-->
@@ -49,11 +49,11 @@
         </geometry>
       </visual>
-      <!--collision name='collision'>
-        <origin xyz="0 0 0" rpy="0 0 0"/>
+      <collision name='collision'>
+        <origin xyz="0.16228 -0.00566 0.1" rpy="0 0 0"/>
         <geometry>
           <mesh filename="package://med_uav_description/meshes/windmill_rotor.dae"
-            scale="1 1 1" />
+            scale="2 2 2" />
         </geometry>
-      </collision-->
+      </collision>
     </link>
     <!--_____________________________________________________________-->

Commit message: Added ground truth odometry sensor.

File: urdf/ardrone.urdf.xacro (robot description, xacro)
@@ -5,4 +5,5 @@
   	<xacro:include filename="$(find med_uav_description)/urdf/ardrone_base.urdf.xacro" />
   	<xacro:include filename="$(find rotors_description)/urdf/component_snippets.xacro" />
+  	<!-- Realistic odometry sensor with noise -->
 	<xacro:odometry_plugin_macro
 		namespace="${namespace}"
@@ -24,4 +25,34 @@
 		noise_normal_linear_velocity="0.0003 0.0003 0.0003"
 		noise_normal_angular_velocity="0.0003 0.0003 0.0003"
+		noise_uniform_position="0.0 0.0 0.0"
+		noise_uniform_quaternion="0.0 0.0 0.0"
+		noise_uniform_linear_velocity="0.0 0.0 0.0"
+		noise_uniform_angular_velocity="0.0 0.0 0.0"
+		enable_odometry_map="false"
+		odometry_map=""
+		image_scale="">
+		<inertia ixx="0.00001" ixy="0.0" ixz="0.0" iyy="0.00001" iyz="0.0" izz="0.00001" /> <!-- [kg m^2] [kg m^2] [kg m^2] [kg m^2] [kg m^2] [kg m^2] -->
+		<origin xyz="0.0 0.0 0.0" rpy="0.0 0.0 0.0" />
+	</xacro:odometry_plugin_macro>
+	<!-- Ground truth odometry sensor without noise -->
+	<xacro:odometry_plugin_macro
+		namespace="${namespace}"
+		odometry_sensor_suffix="gt"
+		parent_link="base_link"
+		pose_topic="pose_gt"
+		pose_with_covariance_topic="pose_with_covariance_gt"
+		position_topic="position_gt"
+		transform_topic="transform_gt"
+		odometry_topic="odometry_gt"
+		parent_frame_id="world"
+		child_frame_id="${namespace}/base_link"
+		mass_odometry_sensor="0.01"
+		measurement_divisor="5"
+		measurement_delay="0"
+		unknown_delay="0.0"
+		noise_normal_position="0.0 0.0 0.0"
+		noise_normal_quaternion="0.0 0.0 0.0"
+		noise_normal_linear_velocity="0.0 0.0 0.0"
+		noise_normal_angular_velocity="0.0 0.0 0.0"
 		noise_uniform_position="0.0 0.0 0.0"
 		noise_uniform_quaternion="0.0 0.0 0.0"

Commit message: added wind parameters to launch file

File: urdf/ardrone.urdf.xacro (robot description, xacro)
@@ -2,4 +2,7 @@
 <robot name="ardrone" xmlns:xacro="http://ros.org/wiki/xacro">
   <xacro:property name="namespace" value="$(arg namespace)" />
+  <xacro:property name="wind_force" value="$(arg wind_force)" />
+  <xacro:property name="wind_start" value="$(arg wind_start)" />
+  <xacro:property name="wind_duration" value="$(arg wind_duration)" />
   <!-- Instantiate ardrone "mechanics" -->
   	<xacro:include filename="$(find med_uav_description)/urdf/ardrone_base.urdf.xacro" />
@@ -77,7 +80,7 @@
 	      <windForceVariance>0.0</windForceVariance>
 	      <windGustDirection>1 1 -0.3</windGustDirection>
-	      <windGustStart>10</windGustStart>
-	      <windGustDuration>10</windGustDuration>
-	      <windGustForceMean>0</windGustForceMean>
+	      <windGustStart>$(arg wind_start)</windGustStart>
+	      <windGustDuration>$(arg wind_duration)</windGustDuration>
+	      <windGustForceMean>$(arg wind_force)</windGustForceMean>
 	      <windGustForceVariance>0</windGustForceVariance>
 	    </plugin>

Commit message: Added wind gust arguments in UAV launch files.

File: urdf/ardrone.urdf.xacro (robot description, xacro)
@@ -5,4 +5,7 @@
   <xacro:property name="wind_start" value="$(arg wind_start)" />
   <xacro:property name="wind_duration" value="$(arg wind_duration)" />
+  <xacro:property name="wind_direction_x" value="$(arg wind_direction_x)" />
+  <xacro:property name="wind_direction_y" value="$(arg wind_direction_y)" />
+  <xacro:property name="wind_direction_z" value="$(arg wind_direction_z)" />
   <!-- Instantiate ardrone "mechanics" -->
   	<xacro:include filename="$(find med_uav_description)/urdf/ardrone_base.urdf.xacro" />
@@ -79,5 +82,5 @@
 	      <windForceMean>0</windForceMean>
 	      <windForceVariance>0.0</windForceVariance>
-	      <windGustDirection>1 1 -0.3</windGustDirection>
+	      <windGustDirection>$(arg wind_direction_x) $(arg wind_direction_y) $(arg wind_direction_z)</windGustDirection>
 	      <windGustStart>$(arg wind_start)</windGustStart>
 	      <windGustDuration>$(arg wind_duration)</windGustDuration>

Commit message: added bebop

File: urdf/ardrone.urdf.xacro (robot description, xacro)
@@ -95,5 +95,5 @@
     <joint name="laser1D_joint" type="fixed">
       <!--<axis xyz="0 0 1" />-->
-      <origin xyz="0.19 0 0.031" rpy="0 0 0"/>
+      <origin xyz="0.111 0 0.0217" rpy="0 0 0"/>
       <parent link="base_link"/>
       <child link="laser1D_link"/>

File: urdf/ardrone_base.urdf.xacro (robot description, xacro)
@@ -3,12 +3,12 @@
   <!-- Properties -->
   <xacro:property name="rotor_velocity_slowdown_sim" value="15" />
-  <xacro:property name="mesh_file" value="ardrone_indoor.dae" />
-  <xacro:property name="mass" value="1.477" />  <!-- [kg] tum_sim 1.477 kg -->
-  <xacro:property name="body_width" value="0.5" /> <!-- [m] old_value 0.1-->
-  <xacro:property name="body_height" value="0.11" /> <!-- [m] -->
+  <xacro:property name="mesh_file" value="bebop.dae" />
+  <xacro:property name="mass" value="0.5" />  <!-- [kg] tum_sim 1.477 kg -->
+  <xacro:property name="body_width" value="0.212" /> <!-- [m] old_value 0.1-->
+  <xacro:property name="body_height" value="0.062" /> <!-- [m] -->
   <xacro:property name="mass_rotor" value="0.01" /> <!-- [kg] -->
-  <xacro:property name="arm_length" value="0.18" /> <!-- [m] -->
-  <xacro:property name="rotor_offset_top" value="0.05" /> <!-- [m] -->
-  <xacro:property name="radius_rotor" value="0.1524" /> <!-- [m] -->
+  <xacro:property name="arm_length" value="0.12905" /> <!-- [m] -->
+  <xacro:property name="rotor_offset_top" value="0.03" /> <!-- [m] -->
+  <xacro:property name="radius_rotor" value="0.0508" /> <!-- [m] -->
   <xacro:property name="motor_constant" value="8.54858e-06" /> <!-- [kg*m/s^2] -->
   <xacro:property name="moment_constant" value="0.016" /> <!-- [m] -->
@@ -62,5 +62,5 @@
     rolling_moment_coefficient="${rolling_moment_coefficient}"
     color="Red">
-    <origin xyz="${cos45*arm_length} ${sin45*arm_length} ${rotor_offset_top}" rpy="0 0 0" />
+    <origin xyz="0.08440513 0.09784210 ${rotor_offset_top}" rpy="0 0 0" />
     <xacro:insert_block name="rotor_inertia" />
   </xacro:vertical_rotor>
@@ -81,5 +81,5 @@
     rolling_moment_coefficient="${rolling_moment_coefficient}"
     color="Red">
-    <origin xyz="${cos45*arm_length} ${-sin45*arm_length} ${rotor_offset_top}" rpy="0 0 0" />
+    <origin xyz="0.08440513 -0.09784210 ${rotor_offset_top}" rpy="0 0 0" />
     <xacro:insert_block name="rotor_inertia" />
   </xacro:vertical_rotor>
@@ -100,5 +100,5 @@
     rolling_moment_coefficient="${rolling_moment_coefficient}"
     color="Blue">
-    <origin xyz="${-cos45*arm_length} ${sin45*arm_length} ${rotor_offset_top}" rpy="0 0 0" />
+    <origin xyz="-0.06853580 0.09784210 ${rotor_offset_top}" rpy="0 0 0" />
     <xacro:insert_block name="rotor_inertia" />
   </xacro:vertical_rotor>
@@ -119,5 +119,5 @@
     rolling_moment_coefficient="${rolling_moment_coefficient}"
     color="Blue">
-    <origin xyz="${-cos45*arm_length} ${-sin45*arm_length} ${rotor_offset_top}" rpy="0 0 0" />
+    <origin xyz="-0.06853580 -0.09784210 ${rotor_offset_top}" rpy="0 0 0" />
     <xacro:insert_block name="rotor_inertia" />
   </xacro:vertical_rotor>

File: urdf/multirotor_base.urdf.xacro (robot description, xacro)
@@ -17,5 +17,5 @@
       </inertial>
       <visual>
-        <origin xyz="0.055 0 0" rpy="0 0 -1.57079632679" />
+        <origin xyz="0 0 0" rpy="0 0 0" />
         <geometry>
           <mesh filename="package://med_uav_description/meshes/${mesh_file}"
@@ -25,5 +25,5 @@
       </visual>
       <collision>
-        <origin xyz="0 0 0.035" rpy="0 0 0" />
+        <origin xyz="0 0 0.0" rpy="0 0 0" />
         <geometry>
           <box size="${body_width} ${body_width} ${body_height}" /> <!-- [m] [m] [m] -->
@@ -79,5 +79,5 @@
           <!-- <cylinder length="0.005" radius="${radius_rotor}"/> --> <!-- [m] -->
           <mesh filename="package://med_uav_description/meshes/propeller_${direction}.dae"
-            scale="0.0008 0.0008 0.0008" />
+            scale="0.00055 0.00055 0.00055" />
           <!-- <box size="${2*radius_rotor} 0.01 0.005"/> -->
         </geometry>
