Commit message: added camera

File: urdf/bebop_base.urdf.xacro (robot description, xacro)
@@ -20,4 +20,5 @@
   <xacro:property name="rotor_drag_coefficient" value="8.06428e-05" />
   <xacro:property name="rolling_moment_coefficient" value="0.000001" />
+  <xacro:property name="PI" value="3.14" />
   <!-- Property Blocks -->
   <xacro:property name="body_inertia">
@@ -125,3 +126,21 @@
     <dampingFactor>0.001</dampingFactor>
   </gazebo>
+  <!-- Camera properties -->
+  <!--xacro:property name="camera_link" value="0.05" />
+  <xacro:property name="camera_inertia">
+    <inertia
+    ixx="1e-12"
+    iyy="1e-12"
+    izz="1e-12"
+    ixy="0.0" ixz="0.0" iyz="0.0" />
+  </xacro:property>
+  <xacro:property name="camera_mass" value="1e-5"/>
+  <xacro:cam
+    namespace="$(arg namespace)"
+    camera_link="${camera_link}"
+    camera_mass="${camera_mass}"
+    parent="base_link">
+    <origin xyz="0.111 0 0.0217" rpy="0 0 0"/>
+    <xacro:insert_block name="camera_inertia"/>
+  </xacro:cam-->
 </robot>

File: urdf/multirotor_base.urdf.xacro (robot description, xacro)
@@ -27,5 +27,5 @@
         <origin xyz="0 0 0.0" rpy="0 0 0" />
         <geometry>
-          <box size="${body_width} ${body_width} ${body_height}" /> <!-- [m] [m] [m] -->
+          <box size="${body_width} ${body_width} ${body_height}" />
         </geometry>
       </collision>
@@ -85,5 +85,5 @@
       <collision>
         <geometry>
-          <cylinder length="0.005" radius="${radius_rotor}" /> <!-- [m] -->
+          <cylinder length="0.005" radius="${radius_rotor}" />
         </geometry>
       </collision>
@@ -111,3 +111,77 @@
     </gazebo>
   </xacro:macro>
+  <!-- Camera macro. Adds a box representing a camera below the UAV
+  @param camera_link Length of the camera box
+  @param camera_mass Mass of the camera
+  @param parent Parent link on which the camera will be fixed
+  @param *origin Block argument defining the origin of the camera with
+  reference to the parent link.
+  @param *inertia Block argument defining camera inertia.
+  -->
+  <xacro:macro name="cam" params="namespace camera_link camera_mass parent *origin *inertia">
+    <!-- Camera link -->
+    <link name="camera_box">
+      <!--collision>
+        <origin xyz="0 0 0" rpy="0 0 0"/>
+        <geometry>
+          <box size="${camera_link} ${camera_link} ${camera_link}"/>
+        </geometry>
+      </collision-->
+      <!--visual>
+        <origin xyz="0 0 0" rpy="0 0 0"/>
+        <geometry>
+          <box size="${camera_link} ${camera_link} ${camera_link}"/>
+        </geometry>
+        <material name="red"/>
+      </visual-->
+      <inertial>
+        <mass value="${camera_mass}" />
+        <origin xyz="0 0 0" rpy="0 0 0"/>
+        <xacro:insert_block name="inertia"/>
+      </inertial>
+    </link>
+    <!-- Camera joint with reference to the parent link -->
+    <joint name="camera_joint" type="fixed">
+      <xacro:insert_block name="origin"/>
+      <parent link="${parent}"/>
+      <child link="camera_box"/>
+    </joint>
+    <!-- camera -->
+    <gazebo reference="camera_box">
+      <sensor type="camera" name="camera1">
+        <update_rate>30.0</update_rate>
+        <camera name="head">
+          <horizontal_fov>1.3962634</horizontal_fov>
+          <image>
+            <width>1920</width>
+            <height>1080</height>
+            <format>R8G8B8</format>
+          </image>
+          <clip>
+            <near>0.02</near>
+            <far>300</far>
+          </clip>
+          <noise>
+            <type>gaussian</type>
+            <mean>0.0</mean>
+            <stddev>0.007</stddev>
+          </noise>
+        </camera>
+        <plugin name="camera_controller" filename="libgazebo_ros_camera.so">
+          <alwaysOn>true</alwaysOn>
+          <updateRate>0.0</updateRate>
+          <cameraName>${namespace}/camera1</cameraName>
+          <imageTopicName>image_raw</imageTopicName>
+          <cameraInfoTopicName>camera_info</cameraInfoTopicName>
+          <frameName>camera_box</frameName>
+          <hackBaseline>0.07</hackBaseline>
+          <distortionK1>0.0</distortionK1>
+          <distortionK2>0.0</distortionK2>
+          <distortionK3>0.0</distortionK3>
+          <distortionT1>0.0</distortionT1>
+          <distortionT2>0.0</distortionT2>
+        </plugin>
+      </sensor>
+    </gazebo>
+  </xacro:macro>
 </robot>

Commit message: added camera

File: urdf/bebop_base.urdf.xacro (robot description, xacro)
@@ -127,5 +127,5 @@
   </gazebo>
   <!-- Camera properties -->
-  <!--xacro:property name="camera_link" value="0.05" />
+  <xacro:property name="camera_link" value="0.05" />
   <xacro:property name="camera_inertia">
     <inertia
@@ -143,4 +143,4 @@
     <origin xyz="0.111 0 0.0217" rpy="0 0 0"/>
     <xacro:insert_block name="camera_inertia"/>
-  </xacro:cam-->
+  </xacro:cam>
 </robot>

File: urdf/multirotor_base.urdf.xacro (robot description, xacro)
@@ -27,5 +27,5 @@
         <origin xyz="0 0 0.0" rpy="0 0 0" />
         <geometry>
-          <box size="${body_width} ${body_width} ${body_height}" />
+          <box size="${body_width} ${body_width} ${body_height}" /> <!-- [m] [m] [m] -->
         </geometry>
       </collision>
@@ -85,5 +85,5 @@
       <collision>
         <geometry>
-          <cylinder length="0.005" radius="${radius_rotor}" />
+          <cylinder length="0.005" radius="${radius_rotor}" /> <!-- [m] -->
         </geometry>
       </collision>

Commit message: changes in body inertia

File: urdf/bebop_base.urdf.xacro (robot description, xacro)
@@ -25,5 +25,5 @@
     <!--inertia ixx="0.00528525" ixy="0.0" ixz="0.0" iyy="0.00528250" iyz="0.0" izz="0.0104" /--> <!-- [kg*m^2] [kg*m^2] [kg*m^2] [kg*m^2] [kg*m^2] [kg*m^2] -->
     <!-- tum_sim -->
-    <inertia ixx="0.01152" ixy="0.0" ixz="0.0" iyy="0.01152" iyz="0.0" izz="0.0218" />
+    <inertia ixx="0.00389" ixy="0.0" ixz="0.0" iyy="0.00389" iyz="0.0" izz="0.0078" />
   </xacro:property>
   <!-- inertia of a single rotor, assuming it is a cuboid. Height=5mm, width=31mm -->
