Commit message: Add velodyne xacro include in bebop.urdf.xacro

File: urdf/bebop.urdf.xacro (robot description, xacro)
@@ -1,4 +1,5 @@
 <?xml version="1.0"?>
 <robot name="bebop" xmlns:xacro="http://ros.org/wiki/xacro">
+  <xacro:property name="enable_velodyne" value="$(arg enable_velodyne)"/>
   <xacro:property name="namespace" value="$(arg namespace)" />
   <xacro:property name="wind_force" value="$(arg wind_force)" />
@@ -137,3 +138,9 @@
 	    </sensor>
   	</gazebo>
+    <xacro:if value="${enable_velodyne}">
+	    <xacro:include filename="$(find velodyne_description)/urdf/VLP-16.urdf.xacro"/>
+	    <VLP-16 parent="base_link" name="velodyne" topic="/velodyne_points" hz="10" samples="440" gpu="false">
+	        <origin xyz="0 0 0.05" rpy="0 0 0" />
+	    </VLP-16>
+    </xacro:if>
 </robot>
